File: h-bridge.kicad_pcb (KiCad board)
At the start: 2 copper layers, 17.8 x 12.6 mm, 12 parts, among them Q1 AO3400A, Q2 AO3400A, Q3 AO3400A, Q4 AO3400A

Commit message: last version
Parts:
- added J1: A, Connector_PinHeader_2.00mm:PinHeader_1x01_P2.00mm_Vertical, F.Cu at (142.5, 84.5)
- added J2: B, Connector_PinHeader_2.00mm:PinHeader_1x01_P2.00mm_Vertical, F.Cu at (125.0, 86.5)
- added J3: M1, Connector_PinHeader_2.00mm:PinHeader_1x01_P2.00mm_Vertical, F.Cu at (133.5, 75.5)
- added J4: M2, Connector_PinHeader_2.00mm:PinHeader_1x01_P2.00mm_Vertical, F.Cu at (138.0, 91.5)
- added J5: GND, Connector_PinHeader_2.00mm:PinHeader_1x01_P2.00mm_Vertical, F.Cu at (125.0, 79.5)
- added J6: 5V, Connector_PinHeader_2.00mm:PinHeader_1x01_P2.00mm_Vertical, F.Cu at (130.0, 91.5)
- moved R1 4.30 mm to (139.5, 83.4)
- moved D3 3.76 mm to (134.7, 79.5), turned to -90 degrees
- moved R4 3.12 mm to (139.5, 87.4)
- moved R3 1.40 mm to (128.5, 85.5)
- moved Q4 0.91 mm to (136.3, 87.4)
- moved R2 0.87 mm to (128.5, 79.5), turned to 90 degrees
- moved D2 0.60 mm to (134.7, 84.5)
Routing:
- net GND: track 6.13 -> 12.9 mm
- net Net-(D1-A): track 13.7 -> 7.11 mm
- net Net-(Q4-G): track 4.44 -> 2.24 mm
- net Net-(D2-A): track 17.1 -> 15.2 mm
- net Net-(Q3-G): track 3.92 -> 2.14 mm
- net Net-(J2-Pin_1): track 5.80 -> 4.18 mm
- net Net-(Q1-G): track 3.81 -> 2.24 mm
- net Net-(J1-Pin_1): track 3.66 -> 2.17 mm
Other:
- board size 17.8 x 12.6 mm -> 14.1 x 12.4 mm
