File: h-bridge.kicad_sch (KiCad schematic)
At the start: 16 parts, among them J1 A, J2 B, J3 M, J4 M2, Q1 AO3400A, Q2 AO3400A, Q3 AO3400A, Q4 AO3400A

Commit message: last version
Parts:
- added J5: GND, Connector_PinHeader_2.00mm:PinHeader_1x01_P2.00mm_Vertical, symbol Connector:Conn_01x01_Pin
- added J6: 5V, Connector_PinHeader_2.00mm:PinHeader_1x01_P2.00mm_Vertical, symbol Connector:Conn_01x01_Pin
- J3: value M -> M1
Connections:
- net +5V: now also J6.1 (Pin_1)
- net GND: now also J5.1 (Pin_1)
